File: Zener.kicad_sch (KiCad schematic)
At the start: 16 parts, among them U2 ADR1399, U3 LT1001

Commit message: Fixed typos
Parts:
- D1: PN BAS116H\,115 -> BAS116H\,115
Changed lines of the file:
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@@
 			)
 		)
-		(property "PN" "BAS116H\\,115 "
+		(property "PN" "BAS116H\\,115"
 			(at 203.2 97.79 0)
 			(hide yes)
