File: reference_board.kicad_pcb (KiCad board)
At the start: 2 copper layers, 34 x 25 mm, 31 parts, among them J1 Conn_02x05_Counter_Clockwise, U1 TMP236, U2 ADR1399, U3 LT1001

Commit message: Replaced stackup table with autogenerated version
Other:
- board text removed: "1.5 mm"
- board text removed: "35 µm"
- board text removed: "Copper"
- board text removed: "Core"
- board text removed: "Material"
- board text removed: "Stackup:"
- board text removed: "Thickness"
